File: imu.kicad_sch (KiCad schematic)
At the start: 3 parts

Commit message: Annotated schematic
Parts:
- gave numbers to parts that had none: 3
Changed lines of the file:
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@@
   (symbol (lib_id "power:GND") (at 114.3 110.49 0) (unit 1)
     (in_bom yes) (on_board yes) (fields_autoplaced)
-    (property "Reference" "#PWR?" (id 0) (at 114.3 116.84 0)
+    (property "Reference" "#PWR011" (id 0) (at 114.3 116.84 0)
       (effects (font (size 1.27 1.27)) hide)
     )
@@
   (symbol (lib_id "power:GND") (at 114.3 91.44 0) (unit 1)
     (in_bom yes) (on_board yes) (fields_autoplaced)
-    (property "Reference" "#PWR?" (id 0) (at 114.3 97.79 0)
+    (property "Reference" "#PWR010" (id 0) (at 114.3 97.79 0)
       (effects (font (size 1.27 1.27)) hide)
     )
@@
   (symbol (lib_id "power:GND") (at 147.32 105.41 0) (unit 1)
     (in_bom yes) (on_board yes) (fields_autoplaced)
-    (property "Reference" "#PWR?" (id 0) (at 147.32 111.76 0)
+    (property "Reference" "#PWR013" (id 0) (at 147.32 111.76 0)
       (effects (font (size 1.27 1.27)) hide)
     )
@@
   (symbol (lib_id "power:+3V3") (at 105.41 86.36 0) (unit 1)
     (in_bom yes) (on_board yes) (fields_autoplaced)
-    (property "Reference" "#PWR?" (id 0) (at 105.41 90.17 0)
+    (property "Reference" "#PWR08" (id 0) (at 105.41 90.17 0)
       (effects (font (size 1.27 1.27)) hide)
     )
@@
   (symbol (lib_id "Device:C_Small") (at 114.3 88.9 0) (unit 1)
     (in_bom yes) (on_board yes)
-    (property "Reference" "C?" (id 0) (at 116.84 88.9062 0)
+    (property "Reference" "C1" (id 0) (at 116.84 88.9062 0)
       (effects (font (size 1.27 1.27)) (justify left))
     )
@@
   (symbol (lib_id "power:GND") (at 147.32 95.25 0) (unit 1)
     (in_bom yes) (on_board yes)
-    (property "Reference" "#PWR?" (id 0) (at 147.32 101.6 0)
+    (property "Reference" "#PWR012" (id 0) (at 147.32 101.6 0)
       (effects (font (size 1.27 1.27)) hide)
     )
@@
   (symbol (lib_id "power:+3V3") (at 105.41 105.41 0) (unit 1)
     (in_bom yes) (on_board yes) (fields_autoplaced)
-    (property "Reference" "#PWR?" (id 0) (at 105.41 109.22 0)
+    (property "Reference" "#PWR09" (id 0) (at 105.41 109.22 0)
       (effects (font (size 1.27 1.27)) hide)
     )
@@
   (symbol (lib_id "IMUs:LSM6DSR") (at 163.83 97.79 0) (unit 1)
     (in_bom yes) (on_board yes) (fields_autoplaced)
-    (property "Reference" "U?" (id 0) (at 163.83 83.82 0))
+    (property "Reference" "U1" (id 0) (at 163.83 83.82 0))
     (property "Value" "LSM6DSR" (id 1) (at 163.83 86.36 0))
     (property "Footprint" "Package_LGA:LGA-14L_3x2.5mm_P0.86mm" (id 2) (at 153.67 91.44 0)
@@
   (symbol (lib_id "Device:C_Small") (at 114.3 107.95 0) (unit 1)
     (in_bom yes) (on_board yes)
-    (property "Reference" "C?" (id 0) (at 116.84 107.9562 0)
+    (property "Reference" "C2" (id 0) (at 116.84 107.9562 0)
       (effects (font (size 1.27 1.27)) (justify left))
     )

Commit message: Added DT connector footprints and began layout
Parts:
- C1, C2: footprint Capacitor_SMD:C_0402_1005Metric -> Capacitor_SMD:C_0603_1608Metric
Changed lines of the file:
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@@
       (effects (font (size 1.27 1.27)) (justify left))
     )
-    (property "Footprint" "Capacitor_SMD:C_0402_1005Metric" (id 2) (at 114.3 88.9 0)
+    (property "Footprint" "Capacitor_SMD:C_0603_1608Metric" (id 2) (at 114.3 88.9 0)
       (effects (font (size 1.27 1.27)) hide)
     )
@@
       (effects (font (size 1.27 1.27)) (justify left))
     )
-    (property "Footprint" "Capacitor_SMD:C_0402_1005Metric" (id 2) (at 114.3 107.95 0)
+    (property "Footprint" "Capacitor_SMD:C_0603_1608Metric" (id 2) (at 114.3 107.95 0)
       (effects (font (size 1.27 1.27)) hide)
     )

Commit message: Created preliminary placement
I hate this
Parts:
- C1, C2: footprint Capacitor_SMD:C_0603_1608Metric -> Capacitor_SMD:C_0603_1608Metric_Pad1.08x0.95mm_HandSolder
Changed lines of the file:
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@@
       (effects (font (size 1.27 1.27)) (justify left))
     )
-    (property "Footprint" "Capacitor_SMD:C_0603_1608Metric" (id 2) (at 114.3 88.9 0)
+    (property "Footprint" "Capacitor_SMD:C_0603_1608Metric_Pad1.08x0.95mm_HandSolder" (id 2) (at 114.3 88.9 0)
       (effects (font (size 1.27 1.27)) hide)
     )
@@
       (effects (font (size 1.27 1.27)) (justify left))
     )
-    (property "Footprint" "Capacitor_SMD:C_0603_1608Metric" (id 2) (at 114.3 107.95 0)
+    (property "Footprint" "Capacitor_SMD:C_0603_1608Metric_Pad1.08x0.95mm_HandSolder" (id 2) (at 114.3 107.95 0)
       (effects (font (size 1.27 1.27)) hide)
     )
