File: vrmsv2.kicad_sch (KiCad schematic)
At the start: 5 parts

Commit message: Created preliminary placement
I hate this
Changed lines of the file:
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@@
   (junction (at 151.13 82.55) (diameter 0) (color 0 0 0 0)
-  )
-  (junction (at 86.36 82.55) (diameter 0) (color 0 0 0 0)
   )
   (junction (at 119.38 82.55) (diameter 0) (color 0 0 0 0)
@@
   )
   (wire (pts (xy 151.13 73.66) (xy 151.13 82.55))
-    (stroke (width 0) (type default) (color 0 0 0 0))
-  )
-  (wire (pts (xy 86.36 82.55) (xy 92.71 82.55))
     (stroke (width 0) (type default) (color 0 0 0 0))
   )
@@
     (stroke (width 0) (type default) (color 0 0 0 0))
   )
-  (wire (pts (xy 85.09 82.55) (xy 86.36 82.55))
-    (stroke (width 0) (type default) (color 0 0 0 0))
-  )
   (wire (pts (xy 100.33 82.55) (xy 104.14 82.55))
     (stroke (width 0) (type default) (color 0 0 0 0))
@@
   )
   (wire (pts (xy 104.14 91.44) (xy 104.14 90.17))
+    (stroke (width 0) (type default) (color 0 0 0 0))
+  )
+  (wire (pts (xy 85.09 82.55) (xy 92.71 82.55))
     (stroke (width 0) (type default) (color 0 0 0 0))
   )
@@
     (pin "1")
   )
-  (symbol (lib_id "power:+24V") (at 86.36 82.55 0) (unit 1)
+  (symbol (lib_id "power:+24V") (at 85.09 82.55 0) (unit 1)
     (in_bom yes) (on_board yes) (fields_autoplaced)
-    (property "Reference" "#PWR040" (id 0) (at 86.36 86.36 0)
+    (property "Reference" "#PWR040" (id 0) (at 85.09 86.36 0)
       (effects (font (size 1.27 1.27)) hide)
     )
-    (property "Value" "+24V" (id 1) (at 86.36 77.47 0))
-    (property "Footprint" "" (id 2) (at 86.36 82.55 0)
+    (property "Value" "+24V" (id 1) (at 85.09 77.47 0))
+    (property "Footprint" "" (id 2) (at 85.09 82.55 0)
       (effects (font (size 1.27 1.27)) hide)
     )
-    (property "Datasheet" "" (id 3) (at 86.36 82.55 0)
+    (property "Datasheet" "" (id 3) (at 85.09 82.55 0)
       (effects (font (size 1.27 1.27)) hide)
     )
